File: TFG_sch.brd (EAGLE design)
At the start: 100 x 80 mm, 23 parts, among them IC1 PIC18F2580-I/SP

Commit message: resistencias
Parts:
- added C2: (no value), rcl:C1206
- added R7: (no value), resistor:R1206
Changed lines of the file:
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@@
 <?xml version="1.0" encoding="utf-8"?>
 <!DOCTYPE eagle SYSTEM "eagle.dtd">
-<eagle version="7.5.0">
+<eagle version="7.4.0">
 <drawing>
 <settings>
@@
 </element>
 <element name="S2" library="switch-misc" package="9077-1" value="9077-1" x="88.9" y="41.91" rot="R90"/>
+<element name="R7" library="resistor" package="R1206" value="" x="2.54" y="-3.81"/>
+<element name="C2" library="rcl" package="C1206" value="" x="2.54" y="-8.89"/>
 </elements>
 <signals>

Commit message: pcb
Parts:
- removed PICKIT: (no value), pinhead:1X06
- removed R1: 100K, resistor-shunt:SMS-0
- removed S1, S2: 9077-1, switch-misc:9077-1
- added C3: 10uF, rcl:C1206
- added D1: 1N5819-T, diode:DO41-7.6
- added JP3: (no value), pinhead:1X02
- added JP4: Vusb, pinhead:1X01
- added JP5: Vcc, pinhead:1X01
- added JP6, JP7: Current Meter, pinhead:1X01
- added LED7: (no value), eagle-ltspice:LED_1206
- added PICKIT3: (no value), pinhead:1X06/90
- added R8: 470, resistor:R1206
- added S3, S4: (no value), switch-omron:B3F-10XX
- added T1: AP1115, zetex:SOT89
- added X1: MINI-USB-UX60-MB-5ST, con-hirose:UX60-MB-5ST
- C1: value (none) -> 10uF; device resistor:C1608 -> rcl:C1206
- C2: value (none) -> 1uF
- LED1, LED2, LED3: value LG_T679-E1F1-1 -> (none); device led:PLCC2 -> eagle-ltspice:LED_1206
- R2, R3, R4, R5, R6: device resistor-shunt:SMS-0 -> resistor:R1206
- R7: value (none) -> 470
- moved R6 65.0 mm to (22.9, 40.6), turned to 270 degrees
- moved C1 49.0 mm to (17.8, 26.7), turned to 270 degrees
- moved LIGH_SENSOR 43.8 mm to (25.4, 57.1), turned to 90 degrees
- moved C2 36.6 mm to (33.0, 11.4), turned to 270 degrees
- moved R7 33.3 mm to (34.3, 6.35), turned to 180 degrees
- moved R2 15.5 mm to (22.9, 33.0), turned to 270 degrees
- moved GROUND_HUMIDITY 9.67 mm to (39.4, 16.5)
- moved R3 8.89 mm to (58.4, 21.6)
- moved R5 8.89 mm to (68.6, 21.6)
- moved ANALOG_SENSOR 6.84 mm to (50.8, 14.0)
- moved LED1 1.27 mm to (58.4, 14.0), turned to 270 degrees
- moved LED3 1.27 mm to (68.6, 14.0), turned to 270 degrees
- turned LED2 to 270 degrees
Connections:
- new net N$34: JP3.1, LED1.C, LED2.C, LED3.C, LED7.C
- new net N$35: LED7.A, R7.1
- new net N$36: D1.A, X1.1
- new net N$37: C3.1, D1.C, R7.2, T1.2, T1.2@1
- new net N$38: JP5.1, JP6.1, PICKIT3.2, R6.1
- new net VO: C1.1, JP4.1, T1.3
- net GND: now also C2.2, C3.2, JP3.2, PICKIT3.3, S3.2, S4.2, T1.1, X1.4, X1.5; no longer LED1.C, LED2.C, LED3.C, PICKIT.3, S1.1, S2.1
- net N$1: now also PICKIT3.1, R2.1, R6.2, S3.4; no longer PICKIT.1, R1.1, R2.2, S1.2
- net N$11: now also R3.2; no longer R5.1
- net N$12: now also R4.2; no longer R4.1
- net N$13: now also R5.2; no longer R3.1
- net N$15: now also PICKIT3.4; no longer PICKIT.4
- net N$16: now also PICKIT3.5; no longer PICKIT.5
- net N$22: now also R8.2; no longer R6.1
- net N$23: now also R2.2; no longer R2.1
- net N$24: now also R8.1, S4.4; no longer R6.2, S2.2
- net N$29: now also PICKIT3.6; no longer PICKIT.6
- net N$31: now also R3.1; no longer R5.2
- net N$32: now also R4.1; no longer R4.2
- net N$33: now also R5.1; no longer R3.2
- net VCC: now also C2.1, JP7.1; no longer C1.1, PICKIT.2, R1.2
Routing:
- net VCC: track 256.9 -> 176.6 mm, vias 1 -> 0
- net N$38: track 0.00 -> 65.1 mm
- net N$16: track 87.8 -> 36.8 mm
- net N$15: track 86.8 -> 36.6 mm
- net N$1: track 90.9 -> 44.0 mm
- net N$19: track 65.7 -> 29.1 mm
- net N$34: track 0.00 -> 28.1 mm
- net N$37: track 0.00 -> 26.5 mm
- net N$26: track 63.7 -> 39.1 mm
- net VO: track 0.00 -> 20.5 mm
- net GND: track 246.2 -> 262.9 mm
- net N$3: track 42.7 -> 27.8 mm, vias 2 -> 0
- net N$24: track 19.7 -> 7.65 mm
- net N$2: track 30.3 -> 22.2 mm
- net N$22: track 39.8 -> 32.6 mm
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- added copper zone on layer 16, net GND
Other:
- board size 100 x 80 mm -> 77.1 x 80 mm
- board text added: "Alejandro García Moreno TFG"
- board text added: "Anag Temp"
- board text added: "Bluetooth"
- board text added: "DHT22"
- board text added: "Diode"
- board text added: "Ground HUM"
- board text added: "LEDs"
- board text added: "Light Sensor"
- board text added: "MiniUSB"
- board text added: "Reset"
- board text added: "Start"
- board text added: "UPC EETAC"
- board text added: "USB USART"
