File: TFG_sch.sch (EAGLE design)
At the start: 25 parts, among them IC1 PIC18F2580-I/SP

Commit message: pcb
Parts:
- removed PICKIT: (no value), pinhead:PINHD-1X6
- removed R1: 100K, resistor-shunt:SMS-0
- removed S1, S2: 9077-1, switch-misc:9077-1
- added C3: 10uF, rcl:C-EUC1206
- added D1: 1N5819-T, diode:1N5819-T
- added JP3: (no value), pinhead:PINHD-1X2
- added JP4: Vusb, pinhead:PINHD-1X1
- added JP5: Vcc, pinhead:PINHD-1X1
- added JP6, JP7: Current Meter, pinhead:PINHD-1X1
- added LED7: (no value), eagle-ltspice:LED_E
- added PICKIT3: (no value), pinhead:PINHD-1X6/90
- added R8: 470, resistor:R-EU_R1206
- added S3, S4: (no value), switch-omron:10-XX
- added T1: AP1115, zetex:NMOSSOT89
- added X1: MINI-USB-UX60-MB-5ST, con-hirose:MINI-USB-UX60-MB-5ST
- C1: value (none) -> 10uF; device resistor:C-USC1608 -> rcl:C-EUC1206
- C2: value (none) -> 1uF
- LED1, LED2, LED3: value LG_T679-E1F1-1 -> (none); device led:LG_T679-E1F1-1 -> eagle-ltspice:LED_E
- R2, R3, R4, R5, R6: device resistor-shunt:SMS-0 -> resistor:R-EU_R1206
- R7: value (none) -> 470
Connections:
- new net N$34: JP3.1, LED1.C, LED2.C, LED3.C, LED7.C
- new net N$35: LED7.A, R7.1
- new net N$36: D1.A, X1.1
- new net N$37: C3.1, D1.C, R7.2, T1.D
- new net N$38: JP5.1, JP6.1, PICKIT3.2, R6.1
- new net VO: C1.1, JP4.1, T1.S
- net GND: now also C2.2, C3.2, JP3.2, PICKIT3.3, S3.S1, S4.S1, T1.G, X1.4, X1.5; no longer LED1.C, LED2.C, LED3.C, PICKIT.3, S1.S, S2.S
- net N$1: now also PICKIT3.1, R2.1, R6.2, S3.P1; no longer PICKIT.1, R1.1, R2.2, S1.P
- net N$11: now also R3.2; no longer R5.1
- net N$12: now also R4.2; no longer R4.1
- net N$13: now also R5.2; no longer R3.1
- net N$15: now also PICKIT3.4; no longer PICKIT.4
- net N$16: now also PICKIT3.5; no longer PICKIT.5
- net N$22: now also R8.2; no longer R6.1
- net N$23: now also R2.2; no longer R2.1
- net N$24: now also R8.1, S4.P1; no longer R6.2, S2.P
- net N$29: now also PICKIT3.6; no longer PICKIT.6
- net N$31: now also R3.1; no longer R5.2
- net N$32: now also R4.1; no longer R4.2
- net N$33: now also R5.1; no longer R3.2
- net VCC: now also C2.1, JP7.1; no longer C1.1, PICKIT.2, R1.2
Other:
- moved on the sheet: C1, C2, LED1, LED3, R3, R5, R6, R7
