File: TFG_sch_V2.brd (EAGLE design)
At the start: 77.1 x 80 mm, 35 parts, among them IC1 PIC18F2580-I/SP, T1 AP1115, X1 MINI-USB-UX60-MB-5ST

Commit message: asd
Parts:
- moved S4 1.27 mm to (73.7, 63.5)
- moved LIGH_SENSOR 1.27 mm to (25.4, 55.9)
Routing:
- net GND: track 261.0 -> 307.9 mm
- net VCC: track 184.4 -> 209.9 mm, vias 0 -> 1
- net N$1: track 44.4 -> 57.7 mm
- net N$38: track 61.6 -> 72.7 mm, vias 0 -> 2
- net N$25: track 34.7 -> 45.6 mm, vias 0 -> 1
- net N$26: track 40.9 -> 48.1 mm
- net N$19: track 29.0 -> 32.1 mm
- net N$18: track 25.1 -> 28.0 mm
- net N$22: track 28.2 -> 30.9 mm
- net N$24: track 6.60 -> 8.82 mm
- net N$34: track 28.3 -> 30.4 mm
- net N$37: track 36.6 -> 38.5 mm
- net N$3: track 27.6 -> 29.1 mm
- net N$28: track 17.4 -> 18.8 mm
- net N$23: track 21.4 -> 22.6 mm
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- added copper zone on layer 16, net GND
- added copper zone on layer 1, net N$14
- removed copper zone on layer 16, net N$14
- removed copper zone on layer 1, net N$30
Other:
- board size 77.1 x 80 mm -> 81 x 80 mm
- board text removed: "Alejandro García Moreno TFG"
- board text removed: "Anag Temp"
- board text removed: "Bluetooth"
- board text removed: "DHT22"
- board text removed: "Diode"
- board text removed: "Ground HUM"
- board text removed: "LEDs"
- board text removed: "Light Sensor"
- board text removed: "MiniUSB"
- board text removed: "Reset"
- board text removed: "Start"
- board text removed: "UPC EETAC"
- board text removed: "USB USART"

Commit message: comint
Parts:
- flipped PICKIT3 to the bottom
Routing:
- net GND: track 307.9 -> 274.8 mm
- net N$1: track 57.7 -> 67.6 mm, vias 0 -> 1
- net N$16: track 37.3 -> 44.2 mm, vias 0 -> 1
- net N$15: track 37.3 -> 41.3 mm
- net N$38: track 72.7 -> 69.6 mm
- net N$18: track 28.0 -> 27.3 mm
Changed lines of the file:
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@@
 <element name="C1" library="rcl" package="C1206" value="10uF" x="16.51" y="24.13" rot="R90"/>
 <element name="JP3" library="pinhead" package="1X02" value="" x="52.07" y="7.62" rot="R90"/>
-<element name="PICKIT3" library="pinhead" package="1X06/90" value="" x="17.78" y="77.47"/>
+<element name="PICKIT3" library="pinhead" package="1X06/90" value="" x="17.78" y="77.47" rot="MR0"/>
 <element name="LED7" library="eagle-ltspice" package="LED_1206" value="" x="41.91" y="6.35">
 <attribute name="SPICEMODEL" value="NONE" x="41.91" y="6.35" size="1.778" layer="27" display="off"/>
@@
 <wire x1="22.7584" y1="34.4932" x2="22.86" y2="34.442" width="0.4064" layer="1"/>
 <wire x1="22.7584" y1="39.116" x2="22.86" y2="39.218" width="0.4064" layer="1"/>
-<wire x1="11.43" y1="54.61" x2="11.43" y2="73.66" width="0.4064" layer="16"/>
 <wire x1="22.86" y1="39.218" x2="20.472" y2="39.218" width="0.4064" layer="1"/>
 <wire x1="20.472" y1="39.218" x2="19.05" y2="40.64" width="0.4064" layer="1"/>
 <wire x1="19.05" y1="40.64" x2="19.05" y2="44.1706" width="0.4064" layer="1"/>
 <wire x1="19.05" y1="44.1706" x2="18.4912" y2="44.7294" width="0.4064" layer="1"/>
-<wire x1="18.4912" y1="44.7294" x2="18.4912" y2="42.6212" width="0.4064" layer="16"/>
-<wire x1="18.4912" y1="42.6212" x2="17.78" y2="41.91" width="0.4064" layer="16"/>
-<wire x1="17.78" y1="41.91" x2="10.16" y2="41.91" width="0.4064" layer="16"/>
-<wire x1="10.16" y1="41.91" x2="8.89" y2="43.18" width="0.4064" layer="16"/>
-<wire x1="8.89" y1="43.18" x2="8.89" y2="52.07" width="0.4064" layer="16"/>
-<wire x1="8.89" y1="52.07" x2="11.43" y2="54.61" width="0.4064" layer="16"/>
+<wire x1="24.13" y1="73.66" x2="24.13" y2="71.12" width="0.4064" layer="16"/>
+<wire x1="24.13" y1="71.12" x2="22.86" y2="69.85" width="0.4064" layer="16"/>
+<wire x1="22.86" y1="69.85" x2="20.32" y2="69.85" width="0.4064" layer="16"/>
+<via x="20.32" y="69.85" extent="1-16" drill="0.6" shape="square"/>
+<wire x1="20.32" y1="69.85" x2="20.32" y2="60.96" width="0.4064" layer="1"/>
+<wire x1="20.32" y1="60.96" x2="19.05" y2="59.69" width="0.4064" layer="1"/>
+<wire x1="19.05" y1="59.69" x2="12.7" y2="59.69" width="0.4064" layer="1"/>
+<wire x1="12.7" y1="59.69" x2="8.89" y2="55.88" width="0.4064" layer="1"/>
+<wire x1="8.89" y1="55.88" x2="8.89" y2="41.91" width="0.4064" layer="1"/>
+<wire x1="8.89" y1="41.91" x2="10.16" y2="40.64" width="0.4064" layer="1"/>
+<wire x1="10.16" y1="40.64" x2="19.05" y2="40.64" width="0.4064" layer="1"/>
 </signal>
 <signal name="N$2">
@@
 <wire x1="36.83" y1="53.34" x2="30.48" y2="59.69" width="0.4064" layer="16"/>
 <wire x1="30.48" y1="59.69" x2="29.21" y2="59.69" width="0.4064" layer="16"/>
-<wire x1="29.21" y1="59.69" x2="19.05" y2="69.85" width="0.4064" layer="16"/>
-<wire x1="19.05" y1="69.85" x2="19.05" y2="73.66" width="0.4064" layer="16"/>
 <wire x1="36.83" y1="50.8" x2="36.83" y2="44.45" width="0.4064" layer="1"/>
+<wire x1="29.21" y1="59.69" x2="22.86" y2="66.04" width="0.4064" layer="16"/>
+<wire x1="22.86" y1="66.04" x2="17.78" y2="66.04" width="0.4064" layer="16"/>
+<wire x1="17.78" y1="66.04" x2="16.51" y2="67.31" width="0.4064" layer="16"/>
+<wire x1="16.51" y1="67.31" x2="16.51" y2="73.66" width="0.4064" layer="16"/>
 </signal>
 <signal name="N$16">
@@
 <wire x1="39.37" y1="53.34" x2="31.75" y2="60.96" width="0.4064" layer="16"/>
 <wire x1="31.75" y1="60.96" x2="30.48" y2="60.96" width="0.4064" layer="16"/>
-<wire x1="30.48" y1="60.96" x2="21.59" y2="69.85" width="0.4064" layer="16"/>
-<wire x1="21.59" y1="69.85" x2="21.59" y2="73.66" width="0.4064" layer="16"/>
 <wire x1="39.37" y1="50.8" x2="39.37" y2="44.45" width="0.4064" layer="1"/>
 <wire x1="39.37" y1="53.34" x2="39.37" y2="50.8" width="0.4064" layer="16"/>
+<wire x1="30.48" y1="60.96" x2="24.13" y2="67.31" width="0.4064" layer="16"/>
+<wire x1="24.13" y1="67.31" x2="19.05" y2="67.31" width="0.4064" layer="16"/>
+<via x="19.05" y="67.31" extent="1-16" drill="0.6" shape="square"/>
+<wire x1="19.05" y1="67.31" x2="17.78" y2="68.58" width="0.4064" layer="1"/>
+<wire x1="13.97" y1="73.66" x2="13.97" y2="71.12" width="0.4064" layer="1"/>
+<wire x1="13.97" y1="71.12" x2="16.51" y2="68.58" width="0.4064" layer="1"/>
+<wire x1="16.51" y1="68.58" x2="17.78" y2="68.58" width="0.4064" layer="1"/>
 </signal>
 <signal name="N$17">
@@
 <contactref element="DHT22" pad="2"/>
 <wire x1="44.45" y1="44.45" x2="44.45" y2="50.8" width="0.4064" layer="1"/>
-<wire x1="44.45" y1="50.8" x2="44.45" y2="55.88" width="0.4064" layer="16"/>
-<wire x1="44.45" y1="55.88" x2="39.37" y2="55.88" width="0.4064" layer="16"/>
 <wire x1="39.37" y1="55.88" x2="33.02" y2="62.23" width="0.4064" layer="16"/>
 <wire x1="33.02" y1="62.23" x2="33.02" y2="64.77" width="0.4064" layer="16"/>
+<wire x1="39.37" y1="55.88" x2="43.18" y2="55.88" width="0.4064" layer="16"/>
+<wire x1="43.18" y1="55.88" x2="44.45" y2="54.61" width="0.4064" layer="16"/>
+<wire x1="44.45" y1="54.61" x2="44.45" y2="50.8" width="0.4064" layer="16"/>
 </signal>
 <signal name="N$19">
@@
 <wire x1="29.21" y1="27.94" x2="26.4668" y2="27.94" width="0.4064" layer="1"/>
 <wire x1="26.4668" y1="27.94" x2="24.13" y2="25.6032" width="0.4064" layer="1"/>
-<wire x1="16.51" y1="73.66" x2="16.51" y2="69.85" width="0.4064" layer="1"/>
 <wire x1="27.94" y1="57.15" x2="25.4" y2="57.15" width="0.4064" layer="1"/>
 <wire x1="34.29" y1="59.69" x2="35.56" y2="60.96" width="0.4064" layer="1"/>
@@
 <wire x1="27.94" y1="57.15" x2="30.48" y2="59.69" width="0.4064" layer="1"/>
 <wire x1="30.48" y1="59.69" x2="34.29" y2="59.69" width="0.4064" layer="1"/>
-<wire x1="25.4" y1="57.15" x2="20.32" y2="57.15" width="0.4064" layer="1"/>
-<wire x1="20.32" y1="57.15" x2="19.05" y2="58.42" width="0.4064" layer="1"/>
-<wire x1="19.05" y1="58.42" x2="19.05" y2="64.77" width="0.4064" layer="1"/>
-<wire x1="19.05" y1="64.77" x2="19.05" y2="67.31" width="0.4064" layer="1"/>
-<wire x1="19.05" y1="67.31" x2="16.51" y2="69.85" width="0.4064" layer="1"/>
-<wire x1="18.4912" y1="49.2506" x2="18.4912" y2="51.3588" width="0.4064" layer="16"/>
-<wire x1="18.4912" y1="51.3588" x2="15.24" y2="54.61" width="0.4064" layer="16"/>
-<wire x1="15.24" y1="54.61" x2="15.24" y2="60.96" width="0.4064" layer="16"/>
-<via x="15.24" y="60.96" extent="1-16" drill="0.6" shape="square"/>
-<wire x1="15.24" y1="60.96" x2="15.24" y2="63.5" width="0.4064" layer="1"/>
-<wire x1="15.24" y1="63.5" x2="16.51" y2="64.77" width="0.4064" layer="1"/>
-<wire x1="16.51" y1="64.77" x2="19.05" y2="64.77" width="0.4064" layer="1"/>
 <wire x1="30.48" y1="13.84" x2="33.15" y2="13.84" width="0.4064" layer="1"/>
 <wire x1="33.15" y1="13.84" x2="34.29" y2="12.7" width="0.4064" layer="1"/>
@@
 <wire x1="25.4" y1="13.97" x2="30.35" y2="13.97" width="0.4064" layer="1"/>
 <wire x1="30.35" y1="13.97" x2="30.48" y2="13.84" width="0.4064" layer="1"/>
-<polygon width="0.4064" layer="16" spacing="5.08" orphans="yes" thermals="no">
+<wire x1="18.4912" y1="49.2506" x2="18.4912" y2="51.3588" width="0.4064" layer="1"/>
+<wire x1="18.4912" y1="51.3588" x2="17.78" y2="52.07" width="0.4064" layer="1"/>
+<wire x1="17.78" y1="52.07" x2="16.51" y2="52.07" width="0.4064" layer="1"/>
+<wire x1="16.51" y1="52.07" x2="15.24" y2="53.34" width="0.4064" layer="1"/>
+<via x="15.24" y="53.34" extent="1-16" drill="0.6" shape="square"/>
+<wire x1="15.24" y1="53.34" x2="15.24" y2="57.15" width="0.4064" layer="16"/>
+<polygon width="0.4064" layer="16">
 <vertex x="6.35" y="80.01"/>
 <vertex x="87.63" y="80.01"/>
@@
 <wire x1="22.86" y1="44.45" x2="22.86" y2="42.062" width="0.4064" layer="1"/>
 <wire x1="24.13" y1="45.72" x2="24.13" y2="48.26" width="0.4064" layer="1"/>
-<wire x1="24.13" y1="48.26" x2="13.97" y2="58.42" width="0.4064" layer="1"/>
-<wire x1="13.97" y1="58.42" x2="13.97" y2="73.66" width="0.4064" layer="1"/>
 <wire x1="10.16" y1="25.4" x2="10.16" y2="30.48" width="0.4064" layer="1"/>
 <wire x1="10.16" y1="30.48" x2="12.7" y2="30.48" width="0.4064" layer="1"/>
@@
 <via x="17.78" y="38.1" extent="1-16" drill="0.6" shape="square"/>
 <wire x1="17.78" y1="38.1" x2="25.4" y2="38.1" width="0.4064" layer="16"/>
+<wire x1="24.13" y1="48.26" x2="21.59" y2="50.8" width="0.4064" layer="1"/>
+<wire x1="21.59" y1="50.8" x2="21.59" y2="73.66" width="0.4064" layer="1"/>
 </signal>
 <signal name="N$14">
-<polygon width="0.4064" layer="1" spacing="5.08">
+<polygon width="0.4064" layer="1">
 <vertex x="6.35" y="80.01"/>
 <vertex x="87.63" y="80.01"/>
-<vertex x="87.63" y="78.74"/>
 <vertex x="87.63" y="0"/>
 <vertex x="6.35" y="0"/>
